Commit message: Converted adroit_door.xml MJCF --> adroit_door.urdf with Gemini 3 Pro - visuals seems more similar to the original compared to codex with gpt-5 conversion

File: my_assets/adroit_door/adroit_door.urdf (robot description, URDF)
Before this commit: robot adroit_door, 3 links, 2 joints
Links:
- removed link door_link
- removed link latch_link
- added link door_panel, mass 2.43; collision box size=0.4 0.1 0.5; visual box size=0.4 0.1 0.5
- added link latch, mass 3.53; collision cylinder length=0.3 radius=0.05; visual cylinder length=0.14 radius=0.04
- added link world
Joints:
- added joint world_to_frame: type fixed, parent world, child frame_link, origin xyz=-0.107339 0.0435293 0.447376 rpy=0 0 0
- joint door_hinge: child door_link -> door_panel; limit lower=0 upper=1.57 effort=50 velocity=2 -> lower=0 upper=1.57 effort=100 velocity=10; origin xyz=0.31 0 0 rpy=0 0 0 -> xyz=0.6 0 0 rpy=0 0 0
- joint latch_joint: child latch_link -> latch; limit lower=0 upper=1.8 effort=30 velocity=5 -> lower=0 upper=1.57 effort=50 velocity=10; origin xyz=-0.15 0 -0.025 rpy=0 0 0 -> xyz=-0.46 0 -0.025 rpy=0 0 0; parent door_link -> door_panel
