Commit message: 1) Extend door height so it almost touches floor 2) door --> no pole, door:hidden - with hiding pole 3) genesis installation instructions

File: my_assets/adroit_door/adroit_door.urdf (robot description, URDF)
Before this commit: robot adroit_door, 4 links, 3 joints
Links:
- link door_panel: geometry collision box size=0.4 0.1 0.897376; visual box size=0.4 0.1 0.897376
- link frame_link: geometry collision cylinder length=0.947376 radius=0.05; collision cylinder length=0.947376 radius=0.05
