Commit message: Touch-guided door pull (Genesis): force pull follows the hinge, slip re-grasp
- touch/pull.py PullController: velocity-regulated force pull, direction re-estimated from
  motion, hinge circle fit, swept angle about the hinge, slip/blocked/end_stop detection
- run_touch_pull impedance loop (compliant lateral + wrist yaw), TOUCH_PULL IPC, api.pull_with_touch
- touch/recovery.py open_with_touch: pull, re-grasp the moved handle (proprio + hinge arc +
  tracking cross-check), resume on the earlier hinge fit; --no-touch -> disabled for A/B
- realism fixes: lever collision, Genesis IK continuity (no branch jumps), finger force 70 N,
  noslip for door scenes
- skill touch-guided-pull, door skill side-grasp note, harness research/touch/door_pull_e2e.py,
  tests/test_touch_pull.py
- A/B: touch 61-62 deg on normal/skew/err/tangent vs open-loop 36 / 9.7 deg

Co-authored-by: Copilot <223556219+Copilot@users.noreply.github.com>

File: my_assets/adroit_door/adroit_door.urdf (robot description, URDF)
Before this commit: robot adroit_door, 4 links, 3 joints
Links:
- link latch: geometry collision cylinder length=0.2 radius=0.02; collision cylinder length=0.3 radius=0.05
