Commit message: Kettle pour end-to-end (physics only), gripper proprioception, tracking review evidence
Kettle "pick up and pour on the microwave" now completes (run 6: plan_completed) with
plain contact physics; the opt-in grasp weld and the SimEnv on_gripper hook are removed.

- GET_ROBOT_STATE reports measured gripper width/holding, eef_pos_at_close,
  max_tilt_since_close and base_pos; prompts say HOLDING/EMPTY instead of "open".
- Reviewer evidence: holding, carried distance since grasp, measured pour tilt/side.
- Planner gets robot_state_after per subtask (measured state beats a false-negative review).
- pour_pose helper + pour-from-held-container skill (near-edge placement, reach cap
  base z + 0.50, re-grasp instead of in-air 180 deg spin).
- Kettle URDF: flat box grip instead of round capsule (holds tilts about the bar axis).
- Hinge-free tracking review evidence (tracking/review_evidence.py), ablation tool + reports.
- Tests: kitchen IPC (hold across boundary, tilt record, base_pos, planner state),
  pour_pose, review evidence.

Co-authored-by: Copilot <223556219+Copilot@users.noreply.github.com>

File: my_assets/franka_kitchen/item_assets/kettle.urdf (robot description, URDF)
Before this commit: robot kettle_urdf, 2 links, 1 joints
Links:
- link kettleroot_1: geometry collision box size=0.2 0.04 0.05; collision box size=0.244 0.244 0.116
- link kettleroot_2: geometry visual box size=0.2 0.04 0.05; visual capsule length=0.03 radius=0.022
