Commit message: insert_key: Genesis turn works (flat collision blade, per-sim plug friction)
- Collision-only 3 mm key blade in 4.4 mm keyway so the key cannot slip past walls
- Plug friction per sim (PyBullet 0.05, Genesis 0.01 N*m frictionloss)
- plans/insert_key.md: status, findings, next steps

Co-authored-by: Copilot <223556219+Copilot@users.noreply.github.com>

File: my_assets/insert_key/key.urdf (robot description, URDF)
Before this commit: robot key, 1 links, 0 joints
Links:
- link key: geometry collision box size=0.01280 0.00300 0.04570; collision box size=0.02400 0.01000 0.01500

File: my_assets/insert_key/lock.urdf (robot description, URDF)
Before this commit: robot lock, 2 links, 1 joints
Links:
- link plug: geometry collision box size=0.00150 0.03600 0.00800; collision box size=0.00150 0.03600 0.00800
